File: Hardware/node_sensor/_restore_backup_2026-06-09T14-44-24-856/node_sensor.kicad_sch (KiCad schematic)
At the start: 15 parts, among them J1 Conn_Jack-DC, J2 Pump, J3 Light, U1 DevKitESP32, U2 DHT11, U3 BH1750, U4 ADS1115, U5 DS3231, U6 Soil-Moisture, U7 Soil-Moisture, U8 Soil-Moisture, U9 Soil-Moisture

Commit message: updated pcb
Connections:
- net GND: no longer U1.32 (GND)
- no-connect marks 36 -> 37
Changed lines of the file:
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@@
+	)
+	(no_connect
+		(at 99.06 58.42)
 	)
 	(no_connect
@@
 		(pts
 			(xy 53.34 134.62) (xy 53.34 140.97)
-		)
-		(stroke
-			(width 0)
-			(type default)
-		)
-	)
-	(wire
-		(pts
-			(xy 99.06 58.42) (xy 102.87 58.42)
 		)
 		(stroke
@@
 					(unit 1)
 				)
-			)
-		)
-	)
-	(symbol
-		(lib_id "MY_SYMBOLS:GND")
-		(at 102.87 58.42 90)
-		(unit 1)
-		(body_style 1)
-		(exclude_from_sim no)
-		(in_bom yes)
-		(on_board yes)
-		(in_pos_files yes)
-		(dnp no)
-		(fields_autoplaced yes)
-		(property "Reference" "#PWR023"
-			(at 109.22 58.42 0)
-			(hide yes)
-			(show_name no)
-			(do_not_autoplace no)
-			(effects
-				(font
-					(size 1.27 1.27)
-				)
-			)
-		)
-		(property "Value" "GND"
-			(at 106.68 58.4199 90)
-			(show_name no)
-			(do_not_autoplace no)
-			(effects
-				(font
-					(size 1.27 1.27)
-				)
-				(justify right)
-			)
-		)
-		(property "Footprint" ""
-			(at 102.87 58.42 0)
-			(hide yes)
-			(show_name no)
-			(do_not_autoplace no)
-			(effects
-				(font
-					(size 1.27 1.27)
-				)
-			)
-		)
-		(property "Datasheet" ""
-			(at 102.87 58.42 0)
-			(hide yes)
-			(show_name no)
-			(do_not_autoplace no)
-			(effects
-				(font
-					(size 1.27 1.27)
-				)
-			)
-		)
-		(property "Description" "Power symbol creates a global label with name \"GND\" , ground"
-			(at 102.87 58.42 0)
-			(hide yes)
-			(show_name no)
-			(do_not_autoplace no)
-			(effects
-				(font
-					(size 1.27 1.27)
-				)
-			)
-		)
-		(pin "1"
-		)
-		(instances
-			(project "node_sensor"
-				(path "/b1f2dde9-9c60-4b08-b31e-edf781363067"
-					(reference "#PWR023")
-					(unit 1)
-				)
