File: Hardware/node_sensor/node_sensor.kicad_sch (KiCad schematic)
At the start: 15 parts, among them J1 Conn_Jack-DC, J2 Pump, J3 Light, U1 DevKitESP32, U2 DHT11, U3 BH1750, U4 ADS1115, U5 DS3231, U6 Soil-Moisture, U7 Soil-Moisture, U8 Soil-Moisture, U9 Soil-Moisture

Commit message: fusion-sensor,check nvs-DB
Connections:
- net +3V3: now also R1.2
- net 1_wire: now also U2.2 (D0)
Other:
- moved on the sheet: R1
Changed lines of the file:
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@@
+	)
+	(junction
+		(at 106.68 147.32)
+		(diameter 0)
+		(color 0 0 0 0)
 	)
 	(junction
@@
 	)
 	(junction
+		(at 100.33 151.13)
+		(diameter 0)
+		(color 0 0 0 0)
+	)
+	(junction
 		(at 45.72 34.29)
 		(diameter 0)
@@
 	(wire
 		(pts
+			(xy 100.33 143.51) (xy 105.41 143.51)
+		)
+		(stroke
+			(width 0)
+			(type default)
+		)
+	)
+	(wire
+		(pts
 			(xy 22.86 34.29) (xy 30.48 34.29)
 		)
@@
 	(wire
 		(pts
+			(xy 100.33 151.13) (xy 109.22 151.13)
+		)
+		(stroke
+			(width 0)
+			(type default)
+		)
+	)
+	(wire
+		(pts
 			(xy 21.59 133.35) (xy 25.4 133.35)
 		)
@@
 	(wire
 		(pts
+			(xy 105.41 147.32) (xy 106.68 147.32)
+		)
+		(stroke
+			(width 0)
+			(type default)
+		)
+	)
+	(wire
+		(pts
 			(xy 57.15 162.56) (xy 59.69 162.56)
 		)
@@
 	(wire
 		(pts
+			(xy 105.41 143.51) (xy 105.41 147.32)
+		)
+		(stroke
+			(width 0)
+			(type default)
+		)
+	)
+	(wire
+		(pts
 			(xy 59.69 116.84) (xy 52.07 116.84)
 		)
@@
 	(wire
 		(pts
-			(xy 102.87 151.13) (xy 109.22 151.13)
-		)
-		(stroke
-			(width 0)
-			(type default)
-		)
-	)
-	(wire
-		(pts
 			(xy 99.06 48.26) (xy 102.87 48.26)
 		)
@@
 	(wire
 		(pts
-			(xy 90.17 151.13) (xy 95.25 151.13)
+			(xy 90.17 151.13) (xy 100.33 151.13)
 		)
 		(stroke
@@
 	(symbol
 		(lib_id "Device:R")
-		(at 99.06 151.13 90)
+		(at 100.33 147.32 180)
 		(unit 1)
 		(body_style 1)
@@
 		(dnp no)
 		(property "Reference" "R1"
-			(at 99.06 148.844 90)
+			(at 98.044 147.32 90)
 			(show_name no)
 			(do_not_autoplace no)
@@
 		)
 		(property "Value" "10K"
-			(at 99.06 153.67 90)
+			(at 102.87 147.32 90)
 			(show_name no)
 			(do_not_autoplace no)
@@
 		)
 		(property "Footprint" "Resistor_THT:R_Axial_DIN0207_L6.3mm_D2.5mm_P10.16mm_Horizontal"
-			(at 99.06 152.908 90)
+			(at 102.108 147.32 90)
 			(hide yes)
 			(show_name no)
@@
 		)
 		(property "Datasheet" ""
-			(at 99.06 151.13 0)
+			(at 100.33 147.32 0)
 			(hide yes)
 			(show_name no)
@@
 		)
 		(property "Description" "Resistor"
-			(at 99.06 151.13 0)
-			(hide yes)
-			(show_name no)
+			(at 100.33 147.32 0)
+			(hide yes)
+			(show_name no)
